File: eagle/projects/multi/crz7shld.brd (EAGLE design)
At the start: 89 x 79 mm, 51 parts, among them IC1 IS62WV51216BLL-55T, J1 HDR-2X6, J2 HDR-2X6, J3 HDR-2X8, J4 HDR-2X3, J5 HDR-2X8, J6 HDR-2X6, J7 HDR-2X6, Q2 BSS138, Q3 BSS138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

Commit message: Order JLCPCB
Parts:
- removed SV3: HEADER, con-lsta:FE08
- removed SV4: HEADER, con-lsta:FE06
- added JP12: ESP32HDR, pinhead2:1X10
- added JP13: LATJTAG, pinhead2:1X08
- added JP14: JUMPER, pinhead2:1X02
- DHT11, JP2, OLED, SR04_0, SR04_1: device pinhead:1X04 -> pinhead2:1X04
- IR: device pinhead:1X03 -> pinhead2:1X03
- JP3: value HEADER -> LATSPI; device pinhead:1X16 -> pinhead2:1X06
- JP5: value HEADER -> ESP32HDR; device pinhead:1X10 -> pinhead2:1X16
- JP8: device pinhead:1X10 -> pinhead2:1X10
- moved JP3 28.4 mm to (77.0, 63.9), turned to 180 degrees
- moved JP5 26.2 mm to (87.0, 37.4)
- moved T2 6.85 mm to (45.2, 20.0)
- moved R2 6.42 mm to (43.9, 23.5)
- moved R9 6.42 mm to (45.8, 23.5)
- moved IR 5.89 mm to (45.1, 15.3), turned to 0 degrees
- moved D1 1.24 mm to (50.1, 20.4)
Connections:
- removed net 5VLAT: JP3.16, JP5.10
- new net N$5: JP12.8, JP14.1
- net GNDLAT: now also JP12.9, JP13.7, JP5.14, JP5.15; no longer JP3.14, JP3.15, JP5.9, SV3.7
- net LSCL: now also JP3.2, JP5.4; no longer JP3.4, SV4.2
- net LSDA: now also JP3.1, JP5.3; no longer JP3.3, SV4.1
- net LSPICK: now also JP3.6; no longer SV4.6
- net LSPICS: now also JP12.2, JP3.3; no longer JP5.2, SV4.3
- net LSPIMI: now also JP3.5; no longer SV4.5
- net LSPIMO: now also JP12.6, JP3.4; no longer JP5.6, SV4.4
- net RX32LAT: now also JP5.11; no longer JP3.11
- net SPICL32: now also JP12.7; no longer JP5.7
- net SPIMI32: now also JP12.4; no longer JP5.4
- net TX32LAT: now also JP5.12; no longer JP3.12
- net VCCLAT: now also JP13.1, JP14.2; no longer JP3.13, JP5.8, SV3.1
Routing:
- net GNDLAT: track 105.8 -> 0.00 mm, vias 1 -> 0
- net SRGND: track 33.4 -> 136.8 mm
- net GND: track 197.4 -> 253.1 mm
- net VCCLAT: track 103.5 -> 67.4 mm, vias 0 -> 1
- net VCC: track 141.9 -> 177.8 mm
- net 5VLAT: track 32.1 -> 0.00 mm
- net SPICL32: track 83.8 -> 65.5 mm
- net N$5: track 0.00 -> 12.1 mm
- net GND2ND: track 9.48 -> 0.00 mm
- net LSPIMO: track 87.5 -> 96.5 mm, vias 1 -> 2
- net SPIMI32: track 61.3 -> 69.0 mm
- net IR_OUT: track 36.6 -> 30.8 mm
- net +5V: track 102.5 -> 96.8 mm
- net LSPICS: track 85.7 -> 89.9 mm, vias 2 -> 1
- net LSPICK: track 47.1 -> 51.0 mm
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- added copper zone on layer 16, net GND
- added copper zone on layer 16, net GND2ND
- added copper zone on layer 16, net GND3RD
- added copper zone on layer 16, net GNDLAT
- removed copper zone on layer 16, net AGND
- removed copper zone on layer 16, net GNDLAT1
- removed copper zone on layer 16, net N$14
- removed copper zone on layer 16, net N$15
Other:
- board text added: "3.3V Source ============== 1: LATTICE/PMOD 0: ESP32 USB (*** CAREFULLY SELECT ***)"
