File: eagle/projects/multi/crz7shld.sch (EAGLE design)
At the start: 51 parts, among them IC1 IS62WV51216BLL-55T, J1 HDR-2X6, J2 HDR-2X6, J3 HDR-2X8, J4 HDR-2X3, J5 HDR-2X8, J6 HDR-2X6, J7 HDR-2X6, Q2 BSS138, Q3 BSS138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

Commit message: Order JLCPCB
Parts:
- removed SV3: HEADER, con-lsta:FE08-1
- removed SV4: HEADER, con-lsta:FE06-1
- added JP12: ESP32HDR, pinhead2:PINHD-1X10
- added JP13: LATJTAG, pinhead2:PINHD-1X8
- added JP14: JUMPER, pinhead2:PINHD-1X2
- DHT11, JP2, OLED, SR04_0, SR04_1: device pinhead:PINHD-1X4 -> pinhead2:PINHD-1X4
- IR: device pinhead:PINHD-1X3 -> pinhead2:PINHD-1X3
- JP3: value HEADER -> LATSPI; device pinhead:PINHD-1X16 -> pinhead2:PINHD-1X6
- JP5: value HEADER -> ESP32HDR; device pinhead:PINHD-1X10 -> pinhead2:PINHD-1X16
- JP8: device pinhead:PINHD-1X10 -> pinhead2:PINHD-1X10
Connections:
- removed net 5VLAT: JP3.16, JP5.10
- new net N$5: JP12.8, JP14.1
- net GNDLAT: now also JP12.9, JP13.7, JP5.14, JP5.15; no longer JP3.14, JP3.15, JP5.9, SV3.7
- net LSCL: now also JP3.2, JP5.4; no longer JP3.4, SV4.2
- net LSDA: now also JP3.1, JP5.3; no longer JP3.3, SV4.1
- net LSPICK: now also JP3.6; no longer SV4.6
- net LSPICS: now also JP12.2, JP3.3; no longer JP5.2, SV4.3
- net LSPIMI: now also JP3.5; no longer SV4.5
- net LSPIMO: now also JP12.6, JP3.4; no longer JP5.6, SV4.4
- net RX32LAT: now also JP5.11; no longer JP3.11
- net SPICL32: now also JP12.7; no longer JP5.7
- net SPIMI32: now also JP12.4; no longer JP5.4
- net TX32LAT: now also JP5.12; no longer JP3.12
- net VCCLAT: now also JP13.1, JP14.2; no longer JP3.13, JP5.8, SV3.1
Other:
- moved on the sheet: ESP01_2, J7
