File: eagle/projects/crz7shld1/cdz7shld1.brd (EAGLE design)
At the start: 100 x 80 mm, 78 parts, among them J1 HDR-2X6, J1FT Header, J2_XME Header, J3 HDR-2X8, J4 HDR-2X3, J5 HDR-2X8, J5G Header, J8 Header, J9 SCREEN, Q1 BSS138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

Commit message: Post build changes.
Parts:
- moved R1 26.9 mm to (70.9, 29.7), turned to 90 degrees
- moved ESP01_3 25.8 mm to (64.5, 27.9)
- moved C1 23.5 mm to (71.6, 24.1), turned to 0 degrees
- renumbered LOLIN to LO, WROVER to WRO
Routing:
- net XGND: track 18.1 -> 201.8 mm
- net TXDESP: track 65.5 -> 35.0 mm
- net RXDESP: track 84.3 -> 55.1 mm
- net X3V: track 187.2 -> 210.4 mm
- net GPO0ESP: track 65.9 -> 45.6 mm, vias 1 -> 0
- net GPO2ESP: track 65.3 -> 47.0 mm, vias 1 -> 0
- net XSDO: track 49.5 -> 54.7 mm
- net CS: track 60.1 -> 56.0 mm
- net CHIP_EN: track 8.52 -> 5.65 mm
- net K5V: track 77.8 -> 76.6 mm

Commit message: wip
Parts:
- moved R18 22.3 mm to (25.0, 35.4), flipped to the bottom
- moved T1 9.76 mm to (25.9, 40.1), flipped to the bottom, turned to 180 degrees
- moved R16 7.73 mm to (12.4, 29.8), flipped to the bottom
- moved R5 6.59 mm to (19.2, 31.5), flipped to the bottom, turned to 180 degrees
- moved Q6 6.39 mm to (20.0, 23.7), flipped to the bottom
- moved R14 5.19 mm to (19.2, 26.2), flipped to the bottom, turned to 180 degrees
- moved C3 4.33 mm to (19.2, 47.9), flipped to the bottom, turned to 90 degrees
- moved Q1 4.08 mm to (14.6, 22.5), flipped to the bottom, turned to 90 degrees
- moved R13 2.99 mm to (19.2, 29.3), flipped to the bottom, turned to 180 degrees
- moved R15 2.95 mm to (14.0, 25.7), flipped to the bottom, turned to 0 degrees
- moved Q5 2.48 mm to (15.5, 29.3), flipped to the bottom, turned to 90 degrees
- moved R4 2.45 mm to (30.1, 38.9), flipped to the bottom, turned to 180 degrees
- moved R17 2.03 mm to (18.1, 20.6), flipped to the bottom, turned to 180 degrees
- moved R19 1.53 mm to (12.8, 40.1), flipped to the bottom, turned to 0 degrees
- moved C1 1.42 mm to (71.6, 22.7), turned to 90 degrees
Connections:
- net ECHOIN: now also J3.8; no longer J3.11
- net GPO0: now also J3.2; no longer J3.6
- net GPO2: now also J3.1; no longer J3.2
- net IRIN: now also J3.6; no longer J3.10
- net SENSIN: now also J3.12; no longer J3.15
- net TRIGOUT: now also J3.10; no longer J3.12
- net URXD: now also J3.4; no longer J3.8
- net UTXD: now also J3.3; no longer J3.4
Routing:
- net K3V: track 115.1 -> 146.8 mm
- net K5V: track 76.6 -> 59.0 mm
- net N$3: track 2.69 -> 19.4 mm
- net IR_OUT: track 47.2 -> 32.7 mm
- net CS: track 56.0 -> 42.2 mm
- net KGND: track 13.4 -> 0.20 mm
- net N$9: track 18.5 -> 5.49 mm
- net TXDESP: track 35.0 -> 45.5 mm, vias 0 -> 1
- net SDO: track 46.1 -> 54.8 mm
- net SENSIN: track 44.8 -> 38.1 mm
- net URXD: track 38.1 -> 32.1 mm
- net GPO0: track 33.4 -> 27.4 mm
- net IROUT: track 41.5 -> 47.1 mm, vias 0 -> 1
- net ECHO: track 16.8 -> 11.3 mm
- net SDI: track 48.9 -> 43.7 mm
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- removed copper zone on layer 1, net K3V
