File: eagle/projects/crz7shld1/cdz7shld1.sch (EAGLE design)
At the start: 78 parts, among them J1 HDR-2X6, J1FT Header, J2_XME Header, J3 HDR-2X8, J4 HDR-2X3, J5 HDR-2X8, J5G Header, J8 Header, J9 SCREEN, Q1 BSS138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

Commit message: Post build changes.
Parts:
- renumbered LOLIN to LO, WROVER to WRO
Changed lines of the file:
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@@
 <setting verticaltext="up"/>
 </settings>
-<grid distance="50" unitdist="mil" unit="mil" style="lines" multiple="1" display="no" altdistance="0.01" altunitdist="inch" altunit="mil"/>
+<grid distance="0.1" unitdist="inch" unit="inch" style="lines" multiple="1" display="no" altdistance="0.01" altunitdist="inch" altunit="inch"/>
 <layers>
 <layer number="1" name="Top" color="4" fill="1" visible="no" active="no"/>
@@
 <part name="ESP01_3" library="pinhead" library_urn="urn:adsk.eagle:library:325" deviceset="PINHD-2X4" device="" package3d_urn="urn:adsk.eagle:package:22461/2" value="ESP01"/>
 <part name="JE1" library="pinhead" library_urn="urn:adsk.eagle:library:325" deviceset="PINHD-2X4" device="" package3d_urn="urn:adsk.eagle:package:22461/2" value="ESP01"/>
-<part name="WROVER" library="pinhead2" deviceset="PINHD-1X4" device="" value="Header"/>
-<part name="LOLIN" library="pinhead2" deviceset="PINHD-1X4" device="" value="Header"/>
+<part name="WRO" library="pinhead2" deviceset="PINHD-1X4" device="" value="Header"/>
+<part name="LO" library="pinhead2" deviceset="PINHD-1X4" device="" value="Header"/>
 <part name="R1" library="rcl" library_urn="urn:adsk.eagle:library:334" deviceset="R-US_" device="R0402" package3d_urn="urn:adsk.eagle:package:23547/3" value="10k"/>
 <part name="R2" library="rcl" library_urn="urn:adsk.eagle:library:334" deviceset="R-US_" device="R0402" package3d_urn="urn:adsk.eagle:package:23547/3" value="10k"/>
@@
 <attribute name="VALUE" x="166.37" y="175.26" size="1.778" layer="96"/>
 </instance>
-<instance part="WROVER" gate="A" x="205.74" y="185.42" smashed="yes">
+<instance part="WRO" gate="A" x="205.74" y="185.42" smashed="yes">
 <attribute name="NAME" x="199.39" y="193.675" size="1.778" layer="95"/>
 <attribute name="VALUE" x="199.39" y="177.8" size="1.778" layer="96"/>
 </instance>
-<instance part="LOLIN" gate="A" x="152.4" y="185.42" smashed="yes" rot="MR0">
+<instance part="LO" gate="A" x="152.4" y="185.42" smashed="yes" rot="MR0">
 <attribute name="NAME" x="151.13" y="193.675" size="1.778" layer="95"/>
 <attribute name="VALUE" x="158.75" y="177.8" size="1.778" layer="96"/>
@@
 <net name="01GND" class="0">
 <segment>
-<pinref part="WROVER" gate="A" pin="1"/>
+<pinref part="WRO" gate="A" pin="1"/>
 <label x="190.5" y="190.5" size="1.778" layer="95"/>
 <pinref part="JE1" gate="A" pin="1"/>
@@
 <wire x1="165.1" y1="190.5" x2="165.1" y2="198.12" width="0.1524" layer="91"/>
 <wire x1="190.5" y1="198.12" x2="190.5" y2="190.5" width="0.1524" layer="91"/>
-<pinref part="LOLIN" gate="A" pin="1"/>
+<pinref part="LO" gate="A" pin="1"/>
 <wire x1="154.94" y1="190.5" x2="165.1" y2="190.5" width="0.1524" layer="91"/>
 <junction x="165.1" y="190.5"/>
@@
 <net name="01TX" class="0">
 <segment>
-<pinref part="WROVER" gate="A" pin="2"/>
+<pinref part="WRO" gate="A" pin="2"/>
 <wire x1="203.2" y1="187.96" x2="187.96" y2="187.96" width="0.1524" layer="91"/>
 <label x="190.5" y="187.96" size="1.778" layer="95"/>
@@
 <wire x1="177.8" y1="190.5" x2="187.96" y2="190.5" width="0.1524" layer="91"/>
 <wire x1="187.96" y1="190.5" x2="187.96" y2="187.96" width="0.1524" layer="91"/>
-<pinref part="LOLIN" gate="A" pin="4"/>
+<pinref part="LO" gate="A" pin="4"/>
 <wire x1="154.94" y1="182.88" x2="154.94" y2="172.72" width="0.1524" layer="91"/>
 <wire x1="154.94" y1="172.72" x2="187.96" y2="172.72" width="0.1524" layer="91"/>
@@
 <net name="01RX" class="0">
 <segment>
-<pinref part="WROVER" gate="A" pin="3"/>
+<pinref part="WRO" gate="A" pin="3"/>
 <label x="190.5" y="185.42" size="1.778" layer="95"/>
 <pinref part="JE1" gate="A" pin="7"/>
@@
 <wire x1="165.1" y1="177.8" x2="182.88" y2="177.8" width="0.1524" layer="91"/>
 <wire x1="182.88" y1="177.8" x2="182.88" y2="185.42" width="0.1524" layer="91"/>
-<pinref part="LOLIN" gate="A" pin="3"/>
+<pinref part="LO" gate="A" pin="3"/>
 <wire x1="154.94" y1="185.42" x2="165.1" y2="185.42" width="0.1524" layer="91"/>
 <wire x1="165.1" y1="185.42" x2="165.1" y2="182.88" width="0.1524" layer="91"/>
@@
 <label x="190.5" y="182.88" size="1.778" layer="95"/>
 <pinref part="JE1" gate="A" pin="8"/>
-<pinref part="LOLIN" gate="A" pin="2"/>
+<pinref part="LO" gate="A" pin="2"/>
 <wire x1="185.42" y1="182.88" x2="177.8" y2="182.88" width="0.1524" layer="91"/>
 <wire x1="154.94" y1="187.96" x2="162.56" y2="187.96" width="0.1524" layer="91"/>
@@
 <wire x1="213.36" y1="175.26" x2="213.36" y2="203.2" width="0.1524" layer="91"/>
 <junction x="185.42" y="175.26"/>
-<pinref part="WROVER" gate="A" pin="4"/>
+<pinref part="WRO" gate="A" pin="4"/>
 <wire x1="185.42" y1="182.88" x2="203.2" y2="182.88" width="0.1524" layer="91"/>
 <junction x="185.42" y="182.88"/>

Commit message: wip
Connections:
- net ECHOIN: now also J3.8; no longer J3.11
- net GPO0: now also J3.2; no longer J3.6
- net GPO2: now also J3.1; no longer J3.2
- net IRIN: now also J3.6; no longer J3.10
- net SENSIN: now also J3.12; no longer J3.15
- net TRIGOUT: now also J3.10; no longer J3.12
- net URXD: now also J3.4; no longer J3.8
- net UTXD: now also J3.3; no longer J3.4
Changed lines of the file:
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@@
 <segment>
 <pinref part="JP4" gate="B" pin="4"/>
-<label x="73.66" y="144.78" size="1.778" layer="95"/>
-<wire x1="91.44" y1="144.78" x2="73.66" y2="144.78" width="0.1524" layer="91"/>
-<pinref part="J3" gate="G$1" pin="12"/>
-<wire x1="73.66" y1="144.78" x2="73.66" y2="149.86" width="0.1524" layer="91"/>
-<wire x1="73.66" y1="149.86" x2="63.5" y2="149.86" width="0.1524" layer="91"/>
+<label x="73.66" y="154.94" size="1.778" layer="95"/>
+<wire x1="91.44" y1="144.78" x2="76.2" y2="144.78" width="0.1524" layer="91"/>
+<pinref part="J3" gate="G$1" pin="10"/>
+<wire x1="63.5" y1="154.94" x2="76.2" y2="154.94" width="0.1524" layer="91"/>
+<wire x1="76.2" y1="154.94" x2="76.2" y2="144.78" width="0.1524" layer="91"/>
 </segment>
 </net>
@@
 <segment>
 <wire x1="91.44" y1="147.32" x2="86.36" y2="147.32" width="0.1524" layer="91"/>
-<wire x1="86.36" y1="147.32" x2="86.36" y2="152.4" width="0.1524" layer="91"/>
 <pinref part="JP4" gate="B" pin="6"/>
-<label x="73.66" y="152.4" size="1.778" layer="95"/>
-<wire x1="63.5" y1="152.4" x2="86.36" y2="152.4" width="0.1524" layer="91"/>
-<pinref part="J3" gate="G$1" pin="11"/>
+<label x="73.66" y="160.02" size="1.778" layer="95"/>
+<wire x1="86.36" y1="160.02" x2="86.36" y2="147.32" width="0.1524" layer="91"/>
+<pinref part="J3" gate="G$1" pin="8"/>
+<wire x1="63.5" y1="160.02" x2="86.36" y2="160.02" width="0.1524" layer="91"/>
 </segment>
 </net>
@@
 <segment>
 <wire x1="91.44" y1="149.86" x2="88.9" y2="149.86" width="0.1524" layer="91"/>
-<wire x1="88.9" y1="149.86" x2="88.9" y2="154.94" width="0.1524" layer="91"/>
 <pinref part="JP4" gate="B" pin="8"/>
-<label x="73.66" y="154.94" size="1.778" layer="95"/>
-<pinref part="J3" gate="G$1" pin="10"/>
-<wire x1="63.5" y1="154.94" x2="88.9" y2="154.94" width="0.1524" layer="91"/>
+<label x="73.66" y="165.1" size="1.778" layer="95"/>
+<wire x1="88.9" y1="165.1" x2="88.9" y2="149.86" width="0.1524" layer="91"/>
+<pinref part="J3" gate="G$1" pin="6"/>
+<wire x1="63.5" y1="165.1" x2="88.9" y2="165.1" width="0.1524" layer="91"/>
 </segment>
 </net>
@@
 <wire x1="99.06" y1="182.88" x2="99.06" y2="193.04" width="0.1524" layer="91"/>
 <wire x1="99.06" y1="193.04" x2="55.88" y2="193.04" width="0.1524" layer="91"/>
-<wire x1="55.88" y1="193.04" x2="55.88" y2="170.18" width="0.1524" layer="91"/>
+<wire x1="55.88" y1="193.04" x2="55.88" y2="172.72" width="0.1524" layer="91"/>
 <label x="73.66" y="193.04" size="1.778" layer="95"/>
+<pinref part="J3" gate="G$1" pin="3"/>
+<wire x1="63.5" y1="172.72" x2="55.88" y2="172.72" width="0.1524" layer="91"/>
+</segment>
+</net>
+<net name="URXD" class="0">
+<segment>
+<pinref part="ESP01" gate="A" pin="8"/>
+<label x="73.66" y="167.64" size="1.778" layer="95"/>
+<wire x1="106.68" y1="167.64" x2="106.68" y2="175.26" width="0.1524" layer="91"/>
 <pinref part="J3" gate="G$1" pin="4"/>
-<wire x1="63.5" y1="170.18" x2="55.88" y2="170.18" width="0.1524" layer="91"/>
-</segment>
-</net>
-<net name="URXD" class="0">
-<segment>
-<pinref part="ESP01" gate="A" pin="8"/>
-<label x="73.66" y="160.02" size="1.778" layer="95"/>
-<wire x1="106.68" y1="160.02" x2="106.68" y2="175.26" width="0.1524" layer="91"/>
-<pinref part="J3" gate="G$1" pin="8"/>
-<wire x1="63.5" y1="160.02" x2="106.68" y2="160.02" width="0.1524" layer="91"/>
+<wire x1="66.04" y1="167.64" x2="106.68" y2="167.64" width="0.1524" layer="91"/>
+<wire x1="63.5" y1="170.18" x2="66.04" y2="170.18" width="0.1524" layer="91"/>
+<wire x1="66.04" y1="170.18" x2="66.04" y2="167.64" width="0.1524" layer="91"/>
 </segment>
 </net>
@@
 <wire x1="114.3" y1="195.58" x2="68.58" y2="195.58" width="0.1524" layer="91"/>
 <label x="73.66" y="195.58" size="1.778" layer="95"/>
-<pinref part="J3" gate="G$1" pin="2"/>
-<wire x1="63.5" y1="175.26" x2="68.58" y2="175.26" width="0.1524" layer="91"/>
-<wire x1="68.58" y1="175.26" x2="68.58" y2="195.58" width="0.1524" layer="91"/>
+<pinref part="J3" gate="G$1" pin="1"/>
+<wire x1="68.58" y1="177.8" x2="68.58" y2="195.58" width="0.1524" layer="91"/>
+<wire x1="63.5" y1="177.8" x2="68.58" y2="177.8" width="0.1524" layer="91"/>
 </segment>
 </net>
@@
 <net name="SENSIN" class="0">
 <segment>
-<pinref part="J3" gate="G$1" pin="15"/>
-<wire x1="63.5" y1="142.24" x2="68.58" y2="142.24" width="0.1524" layer="91"/>
 <pinref part="XDHT11" gate="A" pin="2"/>
 <wire x1="83.82" y1="119.38" x2="68.58" y2="119.38" width="0.1524" layer="91"/>
-<wire x1="68.58" y1="142.24" x2="68.58" y2="119.38" width="0.1524" layer="91"/>
 <label x="68.58" y="116.84" size="1.778" layer="95"/>
+<wire x1="68.58" y1="149.86" x2="68.58" y2="119.38" width="0.1524" layer="91"/>
+<pinref part="J3" gate="G$1" pin="12"/>
+<wire x1="63.5" y1="149.86" x2="68.58" y2="149.86" width="0.1524" layer="91"/>
 </segment>
 </net>
@@
 <pinref part="ESP01" gate="A" pin="6"/>
 <wire x1="106.68" y1="177.8" x2="111.76" y2="177.8" width="0.1524" layer="91"/>
-<wire x1="111.76" y1="177.8" x2="111.76" y2="165.1" width="0.1524" layer="91"/>
-<label x="73.66" y="165.1" size="1.778" layer="95"/>
-<pinref part="J3" gate="G$1" pin="6"/>
-<wire x1="63.5" y1="165.1" x2="86.36" y2="165.1" width="0.1524" layer="91"/>
-<wire x1="86.36" y1="165.1" x2="88.9" y2="165.1" width="0.1524" layer="91"/>
-<wire x1="111.76" y1="165.1" x2="88.9" y2="165.1" width="0.1524" layer="91"/>
-</segment>
-</net>
+<wire x1="111.76" y1="177.8" x2="111.76" y2="170.18" width="0.1524" layer="91"/>
+<label x="73.66" y="170.18" size="1.778" layer="95"/>
+<wire x1="111.76" y1="170.18" x2="68.58" y2="170.18" width="0.1524" layer="91"/>
+<pinref part="J3" gate="G$1" pin="2"/>
+<wire x1="63.5" y1="175.26" x2="68.58" y2="175.26" width="0.1524" layer="91"/>
+<wire x1="68.58" y1="175.26" x2="68.58" y2="170.18" width="0.1524" layer="91"/>
+</segment>
+</net>
