File: eagle/projects/cmod7shld0/crz7shlda0.sch (EAGLE design)
At the start: 26 parts, among them Q1 BSS138, Q2 BSS138, Q3 BSS138, Q4 BSS138

Commit message: cmod7shld0, crz7shlda0 production
Parts:
- removed ESP01: (no value), pinhead:PINHD-2X4
- removed R2: 10k, rcl:R-US_R0402
- added ESP: NA, pinhead:PINHD-2X5
- 3D_ACCEL, IR1, J1, J2, JP0, JP1, PMOD0, SR0, W1_0: value (none) -> NA
- I2C0: value (none) -> I2C
- I2C1: value (none) -> I2Crev
Connections:
- removed net GPO0: ESP01.6, J2.3
- removed net GPO2: ESP01.4, J2.5
- removed net KCHIP_EN: ESP01.3, R2.2
- removed net URST: ESP01.5, J2.4
- removed net URXD: ESP01.8, J2.2
- removed net UTXD: ESP01.1, J2.6
- new net CS_ESP: ESP.1, J2.2
- new net EN_ESP: ESP.4, J2.4
- new net GPIO3: ESP.8, J2.6
- new net GPIO8: ESP.2, J2.3
- new net GPIO9: ESP.6, J2.5
- net K3V: now also ESP.10; no longer ESP01.7, R2.1
- net KGND: now also ESP.9; no longer ESP01.2
- net SPI_CLK: now also ESP.7
- net SPI_MISO: now also ESP.5
- net SPI_MOSI: now also ESP.3
