File: eagle/projects/crz7shlda0/crz7shlda0.sch (EAGLE design)
At the start: 30 parts, among them J3 HDR-2X8, J5 HDR-2X8, Q1 BSS138, Q5 BSS138, Q6 BSS138, T1 MMBT3904

Commit message: cmod7shld0, crz7shlda0 production
Parts:
- removed ESP01: (no value), pinhead:PINHD-2X4
- removed J5: HDR-2X8, Mechanical:HDR-2X8
- removed J5G: (no value), pinhead2:PINHD-1X2
- removed R19: 10k, rcl:R-US_R0402
- added ESP: (no value), pinhead:PINHD-2X5
- I2C: value (none) -> I2C
- I2C2: value (none) -> I2Crev
- JP4: device jumper:JP7Q -> pinhead:PINHD-2X6
- renumbered I2C1 to I2C, J3 to J1, J9 to J2
Connections:
- removed net 3DIRQ: 3D_ACC.8, JP4.7
- removed net GPO0: ESP01.6, J1.2
- removed net GPO2: ESP01.4, J1.1
- removed net KCHIP_EN: ESP01.3, R19.2
- removed net URXD: ESP01.8, J1.4
- removed net UTXD: ESP01.1, J1.3
- new net CS2: ESP.10, J1.4
- new net EN_ESP: ESP.7, J1.2
- new net GPIO3: ESP.3, J1.1
- new net GPIO8: ESP.9, J1.5
- new net GPIO9: ESP.5, J1.3
- net 3D_INT: now also 3D_ACC.8; no longer JP4.8
- net ECHOIN: now also JP4.10; no longer JP4.12
- net ECHO_: now also JP4.9; no longer JP4.11
- net IRIN: now also JP4.12; no longer JP4.14
- net IR_OUT_: now also JP4.11; no longer JP4.13
- net K3V: now also ESP.1; no longer ESP01.7, R19.1
- net KGND: now also ESP.2; no longer ESP01.2, J5G.1, J5G.2
- net SCK: now also ESP.4
- net SDI: now also ESP.6
- net SDO: now also ESP.8
- net TRIGOUT: now also JP4.8; no longer JP4.10
- net TRIG_: now also JP4.7; no longer JP4.9

Commit message: just push latest hanging changes to repo
Parts:
- removed Q1: BSS138, bss138_10:BSS138
- removed R14, R15: 10k, rcl:R-US_R0402
- JP4: device pinhead:PINHD-2X6 -> pinhead:PINHD-2X5
Connections:
- removed net IR_OUT: IR1.1, Q1.D, R14.1
- removed net IR_OUT_: JP4.11, Q1.S, R15.2
- net IRIN: now also IR1.1; no longer JP4.12
- net K3V: now also IR1.3; no longer Q1.G, R15.1
- net K5V: no longer IR1.3, R14.2
Other:
- moved on the sheet: IR1
