File: eagle/projects/esp32md1/esp32md1.brd (EAGLE design)
At the start: 50.2 x 30.8 mm, 13 parts, among them CON3 CON3, CON4 CON4

Commit message: just push latest hanging changes to repo
Parts:
- removed JP4, JP6: I2C2, pinhead2:2X04
- added I2C-I2SMONO: (no value), pinhead2:2X10
- added JGPIO1, JGPIO2: (no value), pinhead2:2X20
- added RPUSCL, RPUSDA: 4.7k, rcl:R0402
- IO: device pinhead2:1X06 -> pinhead2:1X07
- JTAG: value JTAG -> M50-3600542CONN_M50-3600542_HRW-L; device pinhead2:1X06 -> minijtag:CONN_M50-3600542_HRW-L
- moved R3_SDOL 14.5 mm to (41.3, 10.4), turned to 180 degrees
- moved R2_SDOH 11.5 mm to (40.4, 13.2), turned to 0 degrees
- moved R1_CSH 9.82 mm to (41.7, 21.6)
- moved IO 6.35 mm to (15.5, 17.8), turned to 180 degrees
- moved JTAG 4.82 mm to (21.6, 11.5)
Connections:
- net IO35 renamed IO35\
- removed net IO33: JP2.12
- removed net IO34: JP2.10
- removed net IO4: JP1.9
- new net GND3: JGPIO1.12, JGPIO1.30, JGPIO2.12, JGPIO2.30
- new net IO33_BCK: I2C-I2SMONO.9, JP2.12
- new net IO34_DAT: I2C-I2SMONO.11, JP2.10
- new net IO4_WS: I2C-I2SMONO.13, JP1.9
- new net V33Z: JGPIO1.29, JGPIO2.29
- new net V5Z: JGPIO1.11, JGPIO2.11
- net CS: now also CON2.6
- net GND: now also I2C-I2SMONO.10, I2C-I2SMONO.18, I2C-I2SMONO.7, I2C-I2SMONO.8, JTAG.3, JTAG.5; no longer JP4.3, JP4.4, JP6.1, JP6.2, JTAG.2
- net IO0: now also I2C-I2SMONO.15
- net IO18: now also IO.5; no longer IO.3
- net IO19: now also IO.6; no longer IO.4
- net IO2: now also I2C-I2SMONO.17
- net IO21_SDA: now also I2C-I2SMONO.14, I2C-I2SMONO.2, I2C-I2SMONO.3, RPUSDA.2; no longer JP4.7, JP4.8, JP6.7, JP6.8
- net IO22_SCL: now also I2C-I2SMONO.1, I2C-I2SMONO.16, I2C-I2SMONO.4, RPUSCL.2; no longer JP4.5, JP4.6, JP6.5, JP6.6
- net IO23: now also IO.7; no longer IO.5
- net IO26: now also IO.4; no longer IO.6
- net IO5: now also IO.3
- net TCK: now also JTAG.4; no longer JTAG.3
- net TDI: now also JTAG.8; no longer JTAG.5
- net TDO: now also JTAG.6; no longer JTAG.4
- net TMS: now also JTAG.2; no longer JTAG.6
- net VCC: now also I2C-I2SMONO.12, I2C-I2SMONO.19, I2C-I2SMONO.20, I2C-I2SMONO.5, I2C-I2SMONO.6, RPUSCL.1, RPUSDA.1; no longer JP4.1, JP4.2, JP6.3, JP6.4
Routing:
- net V5Z: track 0.00 -> 56.5 mm
- net V33Z: track 0.00 -> 56.5 mm
- net TDI: track 5.94 -> 37.8 mm
- net IO33_BCK: track 0.00 -> 28.2 mm
- net IO34_DAT: track 0.00 -> 26.2 mm
- net IO4_WS: track 0.00 -> 20.3 mm
- net IO26: track 35.1 -> 15.9 mm
- net VCC: track 42.3 -> 58.8 mm
- net TMS: track 35.1 -> 19.2 mm
- net IO0: track 0.00 -> 15.8 mm
- net IO5: track 0.00 -> 15.6 mm
- net SCL_CK: track 20.1 -> 34.7 mm
- net IO23: track 19.4 -> 5.39 mm
- net IO19: track 18.8 -> 6.96 mm
- net IO2: track 0.00 -> 11.3 mm
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- added copper zone on layer 16, net GND3
Other:
- board size 50.2 x 30.8 mm -> 79.3 x 87.6 mm
- board text added: "19 18 26 23 5 16 1"
- board text added: "MISO CS INT2 INT1"
- board text added: "MOSI CLK VCC GND"
- board text added: "SDA SCL VCC GND GND VCC SDA SCL GND VCC SCL SDA VCC GND BCK DAT WS IO0 IO2 VCC"
- board text added: "To Antenna ^^^"
- board text removed: "GND VCC CLK MOSI"
- board text removed: "GND VCC SCL SDA"
- board text removed: "INT1 INT2 CS MISO"
- board text removed: "IO: 26 23 19 18 16 17"
- board text removed: "SDA SCL G V"
- board text removed: "V G TCK TDO TDI TMS"
