File: eagle/projects/esp32md1/esp32md1.sch (EAGLE design)
At the start: 13 parts, among them CON3 CON3, CON4 CON4

Commit message: just push latest hanging changes to repo
Parts:
- removed JP4, JP6: I2C2, pinhead2:PINHD-2X4
- added I2C-I2SMONO: (no value), pinhead2:PINHD-2X10
- added JGPIO1, JGPIO2: (no value), pinhead2:PINHD-2X20
- added RPUSCL, RPUSDA: 4.7k, rcl:R-US_R0402
- IO: device pinhead2:PINHD-1X6 -> pinhead2:PINHD-1X7
- JTAG: value JTAG -> M50-3600542CONN_M50-3600542_HRW-L; device pinhead2:PINHD-1X6 -> minijtag:M50-3600542CONN_M50-3600542_HRW-L
Connections:
- net IO35 renamed IO35\
- removed net IO33: JP2.12
- removed net IO34: JP2.10
- removed net IO4: JP1.9
- new net GND3: JGPIO1.12, JGPIO1.30, JGPIO2.12, JGPIO2.30
- new net IO33_BCK: I2C-I2SMONO.9, JP2.12
- new net IO34_DAT: I2C-I2SMONO.11, JP2.10
- new net IO4_WS: I2C-I2SMONO.13, JP1.9
- new net V33Z: JGPIO1.29, JGPIO2.29
- new net V5Z: JGPIO1.11, JGPIO2.11
- net CS: now also CON2.6
- net GND: now also I2C-I2SMONO.10, I2C-I2SMONO.18, I2C-I2SMONO.7, I2C-I2SMONO.8, JTAG.3, JTAG.5; no longer JP4.3, JP4.4, JP6.1, JP6.2, JTAG.2
- net IO0: now also I2C-I2SMONO.15
- net IO18: now also IO.5; no longer IO.3
- net IO19: now also IO.6; no longer IO.4
- net IO2: now also I2C-I2SMONO.17
- net IO21_SDA: now also I2C-I2SMONO.14, I2C-I2SMONO.2, I2C-I2SMONO.3, RPUSDA.2; no longer JP4.7, JP4.8, JP6.7, JP6.8
- net IO22_SCL: now also I2C-I2SMONO.1, I2C-I2SMONO.16, I2C-I2SMONO.4, RPUSCL.2; no longer JP4.5, JP4.6, JP6.5, JP6.6
- net IO23: now also IO.7; no longer IO.5
- net IO26: now also IO.4; no longer IO.6
- net IO5: now also IO.3
- net TCK: now also JTAG.4; no longer JTAG.3
- net TDI: now also JTAG.8; no longer JTAG.5
- net TDO: now also JTAG.6; no longer JTAG.4
- net TMS: now also JTAG.2; no longer JTAG.6
- net VCC: now also I2C-I2SMONO.12, I2C-I2SMONO.19, I2C-I2SMONO.20, I2C-I2SMONO.5, I2C-I2SMONO.6, RPUSCL.1, RPUSDA.1; no longer JP4.1, JP4.2, JP6.3, JP6.4
Other:
- moved on the sheet: CON1, CON2, CON3, CON4, R1_CSH, R2_SDOH, R3_SDOL
